File: Issue6A.kicad_pcb (KiCad board)
At the start: 2 copper layers, 214 x 130 mm, 218 parts, among them IC1 ULA, IC10 4116, IC11 4116, IC12 4116, IC13 4116, IC14 LM1889, IC15 TMS4532, IC16 TMS4532, IC17 TMS4532, IC18 TMS4532, IC19 TMS4532, IC2 Z80, IC20 TMS4532, IC21 TMS4532, IC22 TMS4532, IC27 ZX8401, IC28 LS04, IC5 ROM, IC6 4116, IC7 4116, IC8 4116, IC9 4116, J1 Conn_02x03_Odd_Even, J2 LKV, J3 LKU, J7 Barrel_Jack_MountingPin, SW1 SW_SPDT, SW2 Optional RESET Switch, T1 Transformer_1P_1S, X1 14Mhz, X2 4.43Mhz

Commit message: Add Gerbers & Updated ibom
Added Gerbers (I still would be wary about getting a PCB made). Updated PCB to change polygons to zones so that the ibom includes them.
Routing:
- net -5V: track 419.4 -> 524.5 mm
- net GND: track 2866.2 -> 2817.9 mm
- net +V_IN: track 49.5 -> 90.7 mm
- net +5V: track 1125.3 -> 1149.3 mm
- added copper zone on F.Cu, net +12VA
- added copper zone on F.Cu, net +5V
- added copper zone on B.Cu, net +V_IN
- added copper zone on B.Cu, net 0V_IN
- added copper zone on B.Cu, net GND
- added copper zone on F.Cu, net GND
